File: task_00.kicad_sch (KiCad schematic)
At the start: 28 parts, among them J1 Screw_Terminal_01x02, 3935700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, J2 Screw_Terminal_01x02, 3935700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, Q1 FQP27P06, U1 TPS54360DDAR

Commit message: Finished with version 0 of the proj
Parts:
- added C12: 47uF, EFVL100ADA470M10B0, Capacitor_SMD:CP_Elec_10x10.5, symbol Device:C
- added C13: 10uF, C3225X7R2A106K250AC, Capacitor_SMD:C_1210_3225Metric_Pad1.33x2.70mm_HandSolder, symbol Device:C
- added D4: SMLVT3V3, SMLVT3V3:DIOM5336X265N, symbol Diode:SMAJ5.0A
- added L2: CDRH104R, CDRH104R:CDRH104R, symbol CDRH104R:CDRH104R
- added R3: 253k, 0603WAF5233T5E, Resistor_SMD:R_0603_1608Metric_Pad0.98x0.95mm_HandSolder, symbol Device:R
- added R4: 84.5k, 0603WAF8452T5E, Resistor_SMD:R_0603_1608Metric_Pad0.98x0.95mm_HandSolder, symbol Device:R
- renumbered C10 to C1, C3 to C10, C9 to C2, C8 to C3, C7 to C4, C1 to C5, C4 to C6, C5 to C7, C2 to C8, C6 to C9, D2 to D1, D3 to D2, D1 to D3, R8 to R1, R1 to R10, R9 to R2, R6 to R5, R3 to R6, R2 to R7, R5 to R8, R7 to R9
Connections:
- net GND: now also D4.2 (A2), R4.2
- net V_OUT: now also D4.1 (A1)
- net VIN: now reaches C1.1, C2.1, C3.1, C4.1, U1.2 (VIN)
- net VIN: now also C13.1, L2.2, R3.1; no longer D2.1 (K), Q1.3
- net EN: now reaches U1.3 (EN)
- net EN: now also R3.2, R4.1
- new net: C12.2, C13.2
- new net VIN_sp: C12.1, D2.1 (K), L2.1, Q1.3
- no-connect marks 2 -> 1
Other:
- moved on the sheet: C1, C10, C11, C2, C3, C4, C5, C6, C7, C8, C9, D1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

Commit message: Version 3
Parts:
- removed U1: TPS54360DDAR, TPS54360DDAR:VREG_LM5017MR_NOPB, symbol New_Library:TPS54360DDAR
- added H1, H2, H3, H4: MountingHole, MountingHole:MountingHole_2.1mm, symbol Mechanical:MountingHole
- added IC1: TPS54360DDAR, SOIC127P600X170-9N, symbol TPS54360DDAR:TPS54360DDAR
- R1: value 10k, RC0603FR-0710KL -> 30, RC0603JR-0730RL
Connections:
- net EN: now also IC1.3 (EN)
- net FB: now also IC1.5 (FB)
- net GND: now also C10.2, C12.2, C13.2, C8.2, D3.2 (A), IC1.7 (GND), IC1.9 (EP)
- net VIN: now also IC1.2 (VIN)
- net at R5.1: now also IC1.4 (RT/CLK)
- net at C5.1: now also IC1.1 (BOOT)
- net at C11.1, C9.1, R6.1: now also IC1.6 (COMP)
- net at C5.2, D3.1 (K), L1.1: now also IC1.8 (SW)
Other:
- moved on the sheet: D4
